File: pcb/dvs.kicad_pcb (KiCad board)
At the start: 2 copper layers, 38.4 x 71.4 mm, 51 parts, among them J1 Conn_02x06_Odd_Even, J2 AudioJack3_Switch, J3 Conn_02x06_Odd_Even, J4 SD_Card_Receptacle, J5 AudioJack3_Switch, U1 MCP6002-xSN

Commit message: feat(pcb): integrate KiCad schematic and PCB layout with audio jack ground fix
- Update pcb/dvs.kicad_sch connecting audio jack sleeve pad to GND.
- Update pcb/dvs.kicad_pcb with updated ground plane routing and trace clearance.
Connections:
- J5 pad S: unconnected-(J5-PadS) -> GND
Changed lines of the file:
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@@
 			(layers "*.Cu" "*.Mask")
 			(remove_unused_layers no)
-			(net "unconnected-(J5-PadS)")
+			(net "GND")
 			(pintype "passive")
 		)
