File: pcb/dvs.kicad_sch (KiCad schematic)
At the start: 51 parts, among them J1 Conn_02x06_Odd_Even, J2 AudioJack3_Switch, J3 Conn_02x06_Odd_Even, J4 SD_Card_Receptacle, J5 AudioJack3_Switch, U1 MCP6002-xSN

Commit message: feat(pcb): integrate KiCad schematic and PCB layout with audio jack ground fix
- Update pcb/dvs.kicad_sch connecting audio jack sleeve pad to GND.
- Update pcb/dvs.kicad_pcb with updated ground plane routing and trace clearance.
Connections:
- net GND: now also J5.S
Changed lines of the file:
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@@
 	(wire
 		(pts
-			(xy 247.65 111.76) (xy 248.92 111.76)
-		)
-		(stroke
-			(width 0)
-			(type default)
-		)
-	)
-	(wire
-		(pts
 			(xy 100.33 111.76) (xy 100.33 116.84)
 		)
@@
 	(wire
 		(pts
+			(xy 245.11 111.76) (xy 248.92 111.76)
+		)
+		(stroke
+			(width 0)
+			(type default)
+		)
+	)
+	(wire
+		(pts
 			(xy 148.59 129.54) (xy 148.59 137.16)
 		)
@@
 	(wire
 		(pts
+			(xy 245.11 106.68) (xy 245.11 111.76)
+		)
+		(stroke
+			(width 0)
+			(type default)
+		)
+	)
+	(wire
+		(pts
 			(xy 242.57 85.09) (xy 242.57 82.55)
 		)
@@
 				)
 			)
+		)
+	)
+	(symbol
+		(lib_id "power:GND")
+		(at 245.11 106.68 180)
+		(unit 1)
+		(body_style 1)
+		(exclude_from_sim no)
+		(in_bom yes)
+		(on_board yes)
+		(in_pos_files yes)
+		(dnp no)
+		(fields_autoplaced yes)
+		(property "Reference" "#PWR031"
+			(at 245.11 100.33 0)
+			(hide yes)
+			(show_name no)
+			(do_not_autoplace no)
+			(effects
+				(font
+					(size 1.27 1.27)
+				)
+			)
+		)
+		(property "Value" "GND"
+			(at 245.11 101.6 0)
+			(show_name no)
+			(do_not_autoplace no)
+			(effects
+				(font
+					(size 1.27 1.27)
+				)
+			)
+		)
+		(property "Footprint" ""
+			(at 245.11 106.68 0)
+			(hide yes)
+			(show_name no)
+			(do_not_autoplace no)
+			(effects
+				(font
+					(size 1.27 1.27)
+				)
+			)
+		)
+		(property "Datasheet" ""
+			(at 245.11 106.68 0)
+			(hide yes)
+			(show_name no)
+			(do_not_autoplace no)
+			(effects
+				(font
+					(size 1.27 1.27)
+				)
+			)
+		)
+		(property "Description" "Power symbol creates a global label with name \"GND\" , ground"
+			(at 245.11 106.68 0)
+			(hide yes)
+			(show_name no)
+			(do_not_autoplace no)
+			(effects
+				(font
+					(size 1.27 1.27)
+				)
+			)
+		)
+		(pin "1"
+		)
+		(instances
+			(project "dvs"
+				(path "/72127889-723a-4a1a-a1d5-6b20fe0a1f96"
+					(reference "#PWR031")
+					(unit 1)
+				)
+			)
